Commit message: 参数调整

File: legged_examples/legged_unitree/legged_unitree_description/urdf/Laika/const.xacro (robot description, xacro)
@@ -56,5 +56,5 @@
     <xacro:property name="trunk_izz" value="0.042827"/>
     <!-- hip (left front) -->
-    <xacro:property name="hip_mass" value="0.16507"/>
+    <xacro:property name="hip_mass" value="0.85"/>   <!-- 0.16507 -->
     <xacro:property name="hip_com_x" value="-0.020153"/>
     <xacro:property name="hip_com_y" value="-0.00047045"/>
