Commit message: d2

File: legged_examples/legged_unitree/urdf_files/leg_urdf20250406_1/urdf/leg_urdf20250406_1.urdf (robot description, URDF)
Before this commit: robot leg_urdf20250406_1, 19 links, 18 joints
Joints:
- removed joint FR_KFE
- added joint RF_KFE: type revolute, parent RF_thigh, child RF_calf, origin xyz=0.024642 -0.0759 -0.28146 rpy=0 0 0, axis 0 -1 0, limit lower=-2.2 upper=0 effort=60 velocity=15

File: legged_examples/legged_unitree/urdf_trans_pkg/common/leg.xacro (robot description, xacro)
@@ -2,159 +2,5 @@
 <robot xmlns:xacro="http://www.ros.org/wiki/xacro">
     <xacro:include filename="$(find legged_unitree_description)/urdf/common/transmission.xacro"/>
-    <xacro:macro name="leg" params="prefix mesh_path mirror mirror_dae front_hind front_hind_dae *origin">
-        <joint name="${prefix}_HAA" type="revolute">
-            <xacro:insert_block name="origin"/>
-            <parent link="base"/>
-            <child link="${prefix}_hip"/>
-            <axis xyz="1 0 0"/>
-            <dynamics damping="${damping}" friction="${friction}"/>
-            <xacro:if value="${(mirror_dae == True)}">
-                <limit effort="${hip_torque_max}" velocity="${hip_velocity_max}" lower="${hip_position_min}"
-                       upper="${hip_position_max}"/>
-            </xacro:if>
-            <xacro:if value="${(mirror_dae == False)}">
-                <limit effort="${hip_torque_max}" velocity="${hip_velocity_max}" lower="${-hip_position_max}"
-                       upper="${-hip_position_min}"/>
-            </xacro:if>
-        </joint>
-        <link name="${prefix}_hip">
-            <visual>
-                <xacro:if value="${(mirror_dae == True) and (front_hind_dae == True)}">
-                    <origin rpy="0 0 0" xyz="0 0 0"/>
-                </xacro:if>
-                <xacro:if value="${(mirror_dae == False) and (front_hind_dae == True)}">
-                    <origin rpy="${pi} 0 0" xyz="0 0 0"/>
-                </xacro:if>
-                <xacro:if value="${(mirror_dae == True) and (front_hind_dae == False)}">
-                    <origin rpy="0 ${pi} 0" xyz="0 0 0"/>
-                </xacro:if>
-                <xacro:if value="${(mirror_dae == False) and (front_hind_dae == False)}">
-                    <origin rpy="${pi} ${pi} 0" xyz="0 0 0"/>
-                </xacro:if>
-                <geometry>
-                    <mesh filename="${mesh_path}/hip.dae"
-                          scale="1 1 1"/>
-                </geometry>
-                <material name="orange"/>
-            </visual>
-            <collision>
-                <origin rpy="${pi/2.0} 0 0" xyz="0 0 0"/>
-                <geometry>
-                    <cylinder length="${hip_length}" radius="${hip_radius}"/>
-                </geometry>
-            </collision>
-            <inertial>
-                <origin rpy="0 0 0" xyz="${hip_com_x*front_hind} ${hip_com_y*mirror} ${hip_com_z}"/>
-                <mass value="${hip_mass}"/>
-                <inertia
-                        ixx="${hip_ixx}" ixy="${hip_ixy*mirror*front_hind}" ixz="${hip_ixz*front_hind}"
-                        iyy="${hip_iyy}" iyz="${hip_iyz*mirror}"
-                        izz="${hip_izz}"/>
-            </inertial>
-        </link>
-        <joint name="${prefix}_HFE" type="revolute">
-            <origin rpy="0 0 0" xyz="0 ${thigh_offset*mirror} 0"/>
-            <parent link="${prefix}_hip"/>
-            <child link="${prefix}_thigh"/>
-            <axis xyz="0 1 0"/>
-            <dynamics damping="${damping}" friction="${friction}"/>
-            <limit effort="${thigh_torque_max}" velocity="${thigh_velocity_max}" lower="${thigh_position_min}"
-                   upper="${thigh_position_max}"/>
-        </joint>
-        <link name="${prefix}_thigh">
-            <visual>
-                <origin rpy="0 0 0" xyz="0 0 0"/>
-                <geometry>
-                    <xacro:if value="${mirror_dae == True}">
-                        <mesh filename="${mesh_path}/thigh.dae"
-                              scale="1 1 1"/>
-                    </xacro:if>
-                    <xacro:if value="${mirror_dae == False}">
-                        <mesh filename="${mesh_path}/thigh_mirror.dae"
-                              scale="1 1 1"/>
-                    </xacro:if>
-                </geometry>
-                <material name="green"/>
-            </visual>
-            <collision>
-                <origin rpy="0 ${pi/2.0+0.1} 0" xyz="${thigh_x_offset} 0 ${-thigh_length/2.0}"/>
-                <geometry>
-                    <box size="${thigh_length} ${thigh_width} ${thigh_height}"/>
-                </geometry>
-            </collision>
-            <collision>
-                <origin rpy="${pi/2.0} 0 0" xyz="0 ${mirror*thigh_shoulder_y_offset} 0"/>
-                <geometry>
-                    <cylinder length="${thigh_shoulder_length}" radius="${thigh_shoulder_radius}"/>
-                </geometry>
-            </collision>
-            <inertial>
-                <origin rpy="0 0 0" xyz="${thigh_com_x} ${thigh_com_y*mirror} ${thigh_com_z}"/>
-                <mass value="${thigh_mass}"/>
-                <inertia
-                        ixx="${thigh_ixx}" ixy="${thigh_ixy*mirror}" ixz="${thigh_ixz}"
-                        iyy="${thigh_iyy}" iyz="${thigh_iyz*mirror}"
-                        izz="${thigh_izz}"/>
-            </inertial>
-        </link>
-        <joint name="${prefix}_KFE" type="revolute">
-            <origin rpy="0 0 0" xyz="0 0 ${-thigh_length}"/>
-            <parent link="${prefix}_thigh"/>
-            <child link="${prefix}_calf"/>
-            <axis xyz="0 1 0"/>
-            <dynamics damping="${damping}" friction="${friction}"/>
-            <limit effort="${calf_torque_max}" velocity="${calf_velocity_max}" lower="${calf_position_min}" upper="${calf_position_max}"/>
-        </joint>
-        <link name="${prefix}_calf">
-            <visual>
-                <origin rpy="0 0 0" xyz="0 0 0"/>
-                <geometry>
-                    <mesh filename="${mesh_path}/calf.dae"
-                          scale="1 1 1"/>
-                </geometry>
-                <material name="blue"/>
-            </visual>
-            <collision>
-                <origin rpy="0 ${pi/2.0} 0" xyz="${calf_x_offset} 0 ${-calf_length/2.0}"/>
-                <geometry>
-                    <box size="${calf_length} ${calf_width} ${calf_height}"/>
-                </geometry>
-            </collision>
-            <inertial>
-                <origin rpy="0 0 0" xyz="${calf_com_x} ${calf_com_y} ${calf_com_z}"/>
-                <mass value="${calf_mass}"/>
-                <inertia
-                        ixx="${calf_ixx}" ixy="${calf_ixy}" ixz="${calf_ixz}"
-                        iyy="${calf_iyy}" iyz="${calf_iyz}"
-                        izz="${calf_izz}"/>
-            </inertial>
-        </link>
-        <joint name="${prefix}_foot_fixed" type="fixed" dont_collapse="true">
-            <origin rpy="0 0 0" xyz="0 0 ${-(calf_length)}"/>
-            <parent link="${prefix}_calf"/>
-            <child link="${prefix}_FOOT"/>
-        </joint>
-        <link name="${prefix}_FOOT">
-            <visual>
-                <origin rpy="0 0 0" xyz="0 0 0"/>
-                <geometry>
-                    <sphere radius="${foot_radius-0.01}"/>
-                </geometry>
-                <material name="red"/>
-            </visual>
-            <collision>
-                <origin rpy="0 0 0" xyz="0 0 0"/>
-                <geometry>
-                    <sphere radius="${foot_radius}"/>
-                </geometry>
-            </collision>
-            <inertial>
-                <mass value="${foot_mass}"/>
-                <inertia
-                        ixx="${(2*foot_mass)/5.0*(foot_radius*foot_radius)}" ixy="0.0" ixz="0.0"
-                        iyy="${(2*foot_mass)/5.0*(foot_radius*foot_radius)}" iyz="0.0"
-                        izz="${(2*foot_mass)/5.0*(foot_radius*foot_radius)}"/>
-            </inertial>
-        </link>
+    <xacro:macro name="leg" params="prefix">
         <gazebo reference="${prefix}_foot_fixed">
             <disableFixedJointLumping>true</disableFixedJointLumping>

File: legged_examples/legged_unitree/urdf_trans_pkg/robot.xacro (robot description, xacro)
@@ -8,4 +8,12 @@
     <xacro:include filename="$(find urdf_trans_pkg)/common/imu.xacro"/>
     <xacro:include filename="$(find leg_urdf20250406_1)/urdf/$(arg urdf_name).urdf" />
-    <xacro:IMU connected_to="base" imu_name="base_imu" xyz="0. 0. 0." rpy="0. 0. 0."/>
+    <!-- <xacro:IMU connected_to="base" imu_name="base_imu" xyz="0. 0. 0." rpy="0. 0. 0."/> -->
+    <!-- <xacro:leg prefix="LF" >
+    </xacro:leg>
+    <xacro:leg prefix="LH" >
+    </xacro:leg>
+    <xacro:leg prefix="RF" >
+    </xacro:leg>
+    <xacro:leg prefix="RH" >
+    </xacro:leg> -->
 </robot>

Commit message: d4.2

File: legged_examples/legged_unitree/urdf_files/leg_urdf20250406_1/urdf/leg_urdf20250406_1.urdf (robot description, URDF)
Before this commit: robot leg_urdf20250406_1, 19 links, 18 joints
Links:
- removed link bae_imu
- added link base_imu, mass 15.8318733004591; collision mesh filename=package://leg_urdf20250406_1/meshes/bae_imu.STL; visual mesh filename=package://leg_urdf20250406_1/meshes/bae_imu.STL

File: legged_examples/legged_unitree/urdf_trans_pkg/robot.xacro (robot description, xacro)
@@ -2,18 +2,18 @@
 <robot xmlns:xacro="http://www.ros.org/wiki/xacro" name="robot">
     <xacro:arg name="robot_type" default="a1"/>
-    <xacro:arg name="urdf_name" default="leg_urdf20250406_1"/>
-    <!-- <xacro:include filename="$(find urdf_trans_pkg)/common/materials.xacro"/> -->
+    <xacro:arg name="urdf_name" default="leg_urdf20250414_1"/>
+    <xacro:include filename="$(find urdf_trans_pkg)/common/materials.xacro"/>
     <xacro:include filename="$(find urdf_trans_pkg)/common/leg.xacro"/>
-    <!-- <xacro:include filename="$(find urdf_trans_pkg)/common/gazebo.xacro"/> -->
+    <xacro:include filename="$(find urdf_trans_pkg)/common/gazebo.xacro"/>
     <!-- <xacro:include filename="$(find urdf_trans_pkg)/common/imu.xacro"/> -->
-    <xacro:include filename="$(find leg_urdf20250406_1)/urdf/$(arg urdf_name).urdf" />
+    <xacro:include filename="$(find leg_urdf20250414_1)/urdf/$(arg urdf_name).urdf" />
     <!-- <xacro:IMU connected_to="base" imu_name="base_imu" xyz="0. 0. 0." rpy="0. 0. 0."/> -->
-    <xacro:leg prefix="LF" >
-    </xacro:leg>
-    <xacro:leg prefix="LH" >
+    <!-- <xacro:leg prefix="LF" >
+    </xacro:leg> -->
+    <!-- <xacro:leg prefix="LH" >
     </xacro:leg>
     <xacro:leg prefix="RF" >
     </xacro:leg>
     <xacro:leg prefix="RH" >
-    </xacro:leg>
+    </xacro:leg> -->
 </robot>
