Commit message: d5.2

File: legged_examples/legged_unitree/urdf_files/leg_urdf20250417_1/urdf/leg_urdf20250417_1.urdf (robot description, URDF)
Before this commit: robot leg_urdf20250417_1, 17 links, 16 joints
Links:
- link LF_FOOT: geometry collision mesh filename=$(find leg_urdf20250417_1)/meshes/LF_FOOT.STL; visual mesh filename=$(find leg_urdf20250417_1)/meshes/LF_FOOT.STL
- link LF_calf: geometry collision mesh filename=$(find leg_urdf20250417_1)/meshes/LF_calf.STL; visual mesh filename=$(find leg_urdf20250417_1)/meshes/LF_calf.STL
- link LF_hip: geometry collision mesh filename=$(find leg_urdf20250417_1)/meshes/LF_hip.STL; visual mesh filename=$(find leg_urdf20250417_1)/meshes/LF_hip.STL
- link LF_thigh: geometry collision mesh filename=$(find leg_urdf20250417_1)/meshes/LF_thigh.STL; visual mesh filename=$(find leg_urdf20250417_1)/meshes/LF_thigh.STL
- link LH_FOOT: geometry collision mesh filename=$(find leg_urdf20250417_1)/meshes/LH_FOOT.STL; visual mesh filename=$(find leg_urdf20250417_1)/meshes/LH_FOOT.STL
- link LH_calf: geometry collision mesh filename=$(find leg_urdf20250417_1)/meshes/LH_calf.STL; visual mesh filename=$(find leg_urdf20250417_1)/meshes/LH_calf.STL
- link LH_hip: geometry collision mesh filename=$(find leg_urdf20250417_1)/meshes/LH_hip.STL; visual mesh filename=$(find leg_urdf20250417_1)/meshes/LH_hip.STL
- link LH_thigh: geometry collision mesh filename=$(find leg_urdf20250417_1)/meshes/LH_thigh.STL; visual mesh filename=$(find leg_urdf20250417_1)/meshes/LH_thigh.STL
- link RF_FOOT: geometry collision mesh filename=$(find leg_urdf20250417_1)/meshes/RF_FOOT.STL; visual mesh filename=$(find leg_urdf20250417_1)/meshes/RF_FOOT.STL
- link RF_calf: geometry collision mesh filename=$(find leg_urdf20250417_1)/meshes/RF_calf.STL; visual mesh filename=$(find leg_urdf20250417_1)/meshes/RF_calf.STL
- link RF_hip: geometry collision mesh filename=$(find leg_urdf20250417_1)/meshes/RF_hip.STL; visual mesh filename=$(find leg_urdf20250417_1)/meshes/RF_hip.STL
- link RF_thigh: geometry collision mesh filename=$(find leg_urdf20250417_1)/meshes/RF_thigh.STL; visual mesh filename=$(find leg_urdf20250417_1)/meshes/RF_thigh.STL
- link RH_FOOT: geometry collision mesh filename=$(find leg_urdf20250417_1)/meshes/RH_FOOT.STL; visual mesh filename=$(find leg_urdf20250417_1)/meshes/RH_FOOT.STL
- link RH_calf: geometry collision mesh filename=$(find leg_urdf20250417_1)/meshes/RH_calf.STL; visual mesh filename=$(find leg_urdf20250417_1)/meshes/RH_calf.STL
- link RH_hip: geometry collision mesh filename=$(find leg_urdf20250417_1)/meshes/RH_hip.STL; visual mesh filename=$(find leg_urdf20250417_1)/meshes/RH_hip.STL
- link RH_thigh: geometry collision mesh filename=$(find leg_urdf20250417_1)/meshes/RH_thigh.STL; visual mesh filename=$(find leg_urdf20250417_1)/meshes/RH_thigh.STL
- link base: geometry collision mesh filename=$(find leg_urdf20250417_1)/meshes/base.STL; visual mesh filename=$(find leg_urdf20250417_1)/meshes/base.STL

Commit message: d5.3

File: legged_examples/legged_unitree/urdf_files/leg_urdf20250417_1/urdf/leg_urdf20250417_1.urdf (robot description, URDF)
Before this commit: robot leg_urdf20250417_1, 17 links, 16 joints
Links:
- link base: geometry collision box size=0.267 0.194 0.114; visual mesh filename=$(find leg_urdf20250417_1)/meshes/base.STL
Joints:
- joint LF_HFE: origin xyz=0.0627 0.0624 0 rpy=0 0 0 -> xyz=0.0627 0.0624 0 rpy=0 1 0
- joint LH_HFE: origin xyz=-0.0632 0.0195 0 rpy=0 0 0 -> xyz=-0.0632 0.0195 0 rpy=0 1 0
- joint RF_HFE: origin xyz=0.0632 -0.0195 0 rpy=0 0 0 -> xyz=0.0632 -0.0195 0 rpy=0 1 0
- joint RH_HFE: origin xyz=-0.04479 -0.037843 0.0022486 rpy=0 0 0 -> xyz=-0.04479 -0.037843 0.0022486 rpy=0 1 0

File: legged_examples/legged_unitree/urdf_trans_pkg/common/gazebo.xacro (robot description, xacro)
@@ -12,5 +12,5 @@
         <plugin name="p3d_base_controller" filename="libgazebo_ros_p3d.so">
             <alwaysOn>true</alwaysOn>
-            <updateRate>1000.0</updateRate>
+            <updateRate>100.0</updateRate>
             <bodyName>base</bodyName>
             <topicName>ground_truth/state</topicName>

Commit message: d7.1 解决rviz不显示的问题

File: legged_examples/legged_unitree/urdf_files/leg_urdf20250417_1/urdf/leg_urdf20250417_1.urdf (robot description, URDF)
Before this commit: robot leg_urdf20250417_1, 17 links, 16 joints
Links:
- link LF_FOOT: geometry collision mesh filename=file:///$(find leg_urdf20250417_1)/meshes/LF_FOOT.STL; visual mesh filename=file:///$(find leg_urdf20250417_1)/meshes/LF_FOOT.STL
- link LF_calf: geometry collision mesh filename=file:///$(find leg_urdf20250417_1)/meshes/LF_calf.STL; visual mesh filename=file:///$(find leg_urdf20250417_1)/meshes/LF_calf.STL
- link LF_hip: geometry collision mesh filename=file:///$(find leg_urdf20250417_1)/meshes/LF_hip.STL; visual mesh filename=file:///$(find leg_urdf20250417_1)/meshes/LF_hip.STL
- link LF_thigh: geometry collision mesh filename=file:///$(find leg_urdf20250417_1)/meshes/LF_thigh.STL; visual mesh filename=file:///$(find leg_urdf20250417_1)/meshes/LF_thigh.STL
- link LH_FOOT: geometry collision mesh filename=file:///$(find leg_urdf20250417_1)/meshes/LH_FOOT.STL; visual mesh filename=file:///$(find leg_urdf20250417_1)/meshes/LH_FOOT.STL
- link LH_calf: geometry collision mesh filename=file:///$(find leg_urdf20250417_1)/meshes/LH_calf.STL; visual mesh filename=file:///$(find leg_urdf20250417_1)/meshes/LH_calf.STL
- link LH_hip: geometry collision mesh filename=file:///$(find leg_urdf20250417_1)/meshes/LH_hip.STL; visual mesh filename=file:///$(find leg_urdf20250417_1)/meshes/LH_hip.STL
- link LH_thigh: geometry collision mesh filename=file:///$(find leg_urdf20250417_1)/meshes/LH_thigh.STL; visual mesh filename=file:///$(find leg_urdf20250417_1)/meshes/LH_thigh.STL
- link RF_FOOT: geometry collision mesh filename=file:///$(find leg_urdf20250417_1)/meshes/RF_FOOT.STL; visual mesh filename=file:///$(find leg_urdf20250417_1)/meshes/RF_FOOT.STL
- link RF_calf: geometry collision mesh filename=file:///$(find leg_urdf20250417_1)/meshes/RF_calf.STL; visual mesh filename=file:///$(find leg_urdf20250417_1)/meshes/RF_calf.STL
- link RF_hip: geometry collision mesh filename=file:///$(find leg_urdf20250417_1)/meshes/RF_hip.STL; visual mesh filename=file:///$(find leg_urdf20250417_1)/meshes/RF_hip.STL
- link RF_thigh: geometry collision mesh filename=file:///$(find leg_urdf20250417_1)/meshes/RF_thigh.STL; visual mesh filename=file:///$(find leg_urdf20250417_1)/meshes/RF_thigh.STL
- link RH_FOOT: geometry collision mesh filename=file:///$(find leg_urdf20250417_1)/meshes/RH_FOOT.STL; visual mesh filename=file:///$(find leg_urdf20250417_1)/meshes/RH_FOOT.STL
- link RH_calf: geometry collision mesh filename=file:///$(find leg_urdf20250417_1)/meshes/RH_calf.STL; visual mesh filename=file:///$(find leg_urdf20250417_1)/meshes/RH_calf.STL
- link RH_hip: geometry collision mesh filename=file:///$(find leg_urdf20250417_1)/meshes/RH_hip.STL; visual mesh filename=file:///$(find leg_urdf20250417_1)/meshes/RH_hip.STL
- link RH_thigh: geometry collision mesh filename=file:///$(find leg_urdf20250417_1)/meshes/RH_thigh.STL; visual mesh filename=file:///$(find leg_urdf20250417_1)/meshes/RH_thigh.STL
- link base: geometry collision mesh filename=file:///$(find leg_urdf20250417_1)/meshes/base.STL; visual mesh filename=file:///$(find leg_urdf20250417_1)/meshes/base.STL

Commit message: d8 可以站立了，trot还会摔倒

File: legged_examples/legged_unitree/urdf_files/leg_urdf20250417_1/urdf/leg_urdf20250417_1.urdf (robot description, URDF)
Before this commit: robot leg_urdf20250417_1, 17 links, 16 joints
Links:
- link LF_FOOT: geometry collision sphere radius=0.02; visual mesh filename=file:///$(find leg_urdf20250417_1)/meshes/LF_FOOT.STL
- link LH_FOOT: geometry collision sphere radius=0.02; visual mesh filename=file:///$(find leg_urdf20250417_1)/meshes/LH_FOOT.STL
- link RF_FOOT: geometry collision sphere radius=0.02; visual mesh filename=file:///$(find leg_urdf20250417_1)/meshes/RF_FOOT.STL
- link RH_FOOT: geometry collision sphere radius=0.02; visual mesh filename=file:///$(find leg_urdf20250417_1)/meshes/RH_FOOT.STL
- link base: geometry collision box size=0.41 0.23 0.137; visual mesh filename=file:///$(find leg_urdf20250417_1)/meshes/base.STL

Commit message: d9 发现问题了，屏蔽了大腿和小腿的碰撞后可trot

File: legged_examples/legged_unitree/urdf_files/leg_urdf20250417_1/urdf/leg_urdf20250417_1.urdf (robot description, URDF)
Before this commit: robot leg_urdf20250417_1, 17 links, 16 joints
Links:
- link LF_calf: geometry visual mesh filename=file:///$(find leg_urdf20250417_1)/meshes/LF_calf.STL
- link LF_thigh: geometry visual mesh filename=file:///$(find leg_urdf20250417_1)/meshes/LF_thigh.STL
- link LH_calf: geometry visual mesh filename=file:///$(find leg_urdf20250417_1)/meshes/LH_calf.STL
- link LH_thigh: geometry visual mesh filename=file:///$(find leg_urdf20250417_1)/meshes/LH_thigh.STL
- link RF_calf: geometry visual mesh filename=file:///$(find leg_urdf20250417_1)/meshes/RF_calf.STL
- link RF_thigh: geometry visual mesh filename=file:///$(find leg_urdf20250417_1)/meshes/RF_thigh.STL
- link RH_calf: geometry visual mesh filename=file:///$(find leg_urdf20250417_1)/meshes/RH_calf.STL
- link RH_thigh: geometry visual mesh filename=file:///$(find leg_urdf20250417_1)/meshes/RH_thigh.STL
